File: button timer v1.2_[Coin_Cell&LIPO]/button timer v1.2.kicad_pcb (KiCad board)
At the start: 2 copper layers, 21 x 51.6 mm, 27 parts, among them J1 Conn_01x05_Female, SW1 SW_Push, SW2 SW_Push, U1 TPS61097A, U2 AP2112K-3.3, U3 TPL5111, X1 ESP-12E

Commit message: 23.02 00:40
Other:
- board text added: "LK"

Commit message: 23.02 13:31
Parts:
- added C5: 100nF, handsolder:C_0805_2012handsodermod, B.Cu at (126.5, 51.8)
- C4: footprint handsolder:C_0402_1005Metric_Pad0.74x0.62mm_HandSoldermod -> Capacitor_SMD:C_0402_1005Metric_Pad0.74x0.62mm_HandSolder
Routing:
- net /GND: track 120.7 -> 123.4 mm
- net Net-(BT1-Pad1): track 44.9 -> 47.1 mm
