File: button timer v1.2_[Coin_Cell&LIPO]/button timer v1.2.sch (KiCad schematic (older format))
At the start: 27 parts, among them J1 Conn_01x05_Female, SW1 SW_Push, SW2 SW_Push, U1 TPS61097A, U2 AP2112K-3.3, U3 TPL5111, X1 ESP-12E

Commit message: 23.02 13:31
Parts:
- added C5: 100nF, handsolder:C_0805_2012handsodermod, symbol Device:C
- X1: footprint RF_Module:ESP-12E -> handsolder:ESP-12Elesssilk
Connections:
- net GND: now also C5.2
- net at BT1.1 (+), BT2.1 (+), C1.2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: now also C5.1
Changed lines of the file:
@@
 F 0 "X1" H 6000 3400 50  0001 C CNN
 F 1 "ESP-12E" H 6000 3400 50  0001 C CNN
-F 2 "RF_Module:ESP-12E" H 6000 3400 50  0001 C CNN
+F 2 "handsolder:ESP-12Elesssilk" H 6000 3400 50  0001 C CNN
 F 3 "" H 6000 3400 50  0001 C CNN
 	1    6000 3400
@@
 GND
 Wire Wire Line
-	2550 4150 2550 5050
+	2550 4150 2550 4900
 Wire Wire Line
 	2550 5050 2250 5050
@@
 Text Label 2750 6550 3    50   ~ 0
 GND
+$Comp
+L Device:C C5
+U 1 1 6034F848
+P 2400 4900
+F 0 "C5" V 2148 4900 50  0000 C CNN
+F 1 "100nF" V 2239 4900 50  0000 C CNN
+F 2 "handsolder:C_0805_2012handsodermod" H 2438 4750 50  0001 C CNN
+F 3 "~" H 2400 4900 50  0001 C CNN
+	1    2400 4900
+	0    1    1    0
+$EndComp
+Connection ~ 2550 4900
+Wire Wire Line
+	2550 4900 2550 5050
+Text Label 2250 4900 2    50   ~ 0
+GND
 $EndSCHEMATC
