File: button timer v1.2_[Coin_Cell&LIPO][TPL5110]/button timer v1.2_[Coin_Cell&LIPO][TPL5110].sch (KiCad schematic (older format))
At the start: 27 parts, among them J1 Conn_01x05_Female, Q1 TSM2301ACX, SW1 SW_Push, SW2 SW_Push, U1 TPS61097A, U2 AP2112K-3.3, U3 TPL5110, X1 ESP-12E

Commit message: 3D Models etwas verbessert
Parts:
- J1: footprint Connector_PinHeader_2.54mm:PinHeader_1x05_P2.54mm_Vertical -> handsolder:PinSocket_1x05_P2.54mm_Vertical_mod
- SW1: footprint Button_Switch_THT:SW_PUSH_6mm -> handsolder:SW_PUSH_6mm_H8mm_mod
- SW2: footprint Button_Switch_SMD:SW_SPST_EVQPE1 -> handsolder:SW_SPST_B3U-1000P_mod
Changed lines of the file:
@@
 F 0 "SW2" H 7800 2335 50  0000 C CNN
 F 1 "SW_Push" H 7800 2244 50  0000 C CNN
-F 2 "Button_Switch_SMD:SW_SPST_EVQPE1" H 7800 2250 50  0001 C CNN
+F 2 "handsolder:SW_SPST_B3U-1000P_mod" H 7800 2250 50  0001 C CNN
 F 3 "~" H 7800 2250 50  0001 C CNN
 	1    7800 2050
@@
 F 0 "SW1" H 1100 5935 50  0000 C CNN
 F 1 "SW_Push" H 1100 5844 50  0000 C CNN
-F 2 "Button_Switch_THT:SW_PUSH_6mm" H 1100 5850 50  0001 C CNN
+F 2 "handsolder:SW_PUSH_6mm_H8mm_mod" H 1100 5850 50  0001 C CNN
 F 3 "~" H 1100 5850 50  0001 C CNN
 	1    1100 5650
@@
 F 0 "J1" H 8328 3576 50  0000 L CNN
 F 1 "Conn_01x05_Female" H 8328 3485 50  0000 L CNN
-F 2 "Connector_PinHeader_2.54mm:PinHeader_1x05_P2.54mm_Vertical" H 8300 3550 50  0001 C CNN
+F 2 "handsolder:PinSocket_1x05_P2.54mm_Vertical_mod" H 8300 3550 50  0001 C CNN
 F 3 "~" H 8300 3550 50  0001 C CNN
 	1    8300 3550
