File: button_timer v1.2.1_Coin_Cell[TPL5111]/button timer v1.2.1_Coin_Cell.sch (KiCad schematic (older format))
At the start: 25 parts, among them J1 Conn_01x05_Female, Q1 TSM2323, SW1 SW_Push, SW2 SW_Push, U1 TPS61097A, U2 TPL5110, X1 ESP-12E

Commit message: :rocket: :full_moon_with_face:
Parts:
- removed Q1: TSM2323, Package_TO_SOT_SMD:SOT-23, symbol Transistor_FET:TSM2301ACX
- removed U2: TPL5110, Package_TO_SOT_SMD:SOT-23-6, symbol Timer:TPL5110
- added U3: TPL5111, handsolder:SOT-23-6handsoldering, symbol button-timer-v1.2.1_Coin_Cell-rescue:TPL5111-Timer-button-timer-rescue-button-t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
Connections:
- net GND: now also U3.2 (GND), U3.6 (EN/ONE_SHOT)
- net GPIO4: now also U3.4 (DONE)
- net at BT1.1 (+), C1.2, C5.2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: now also L1.1, U1.1 (VIN), U3.1 (VDD)
- net at R6.2, R8.2, SW1.2: now also U3.3 (DELAY/M_DRV)
- net at R7.1: now also U3.5 (~DRV); no longer U1.3 (EN)
- new net: R7.2, U1.3 (EN)
Other:
- moved on the sheet: C3, L1, R7, U1
Changed lines of the file:
@@
 Wire Wire Line
 	1300 5750 1300 5650
+$Comp
+L button-timer-v1.2.1_Coin_Cell-rescue:TPL5111-Timer-button-timer-rescue-button-timer-v1.2-rescue-button-timer-v1.2-rescue U3
+U 1 1 6031B6A7
+P 2250 5650
+F 0 "U3" H 2200 6331 50  0000 C CNN
+F 1 "TPL5111" H 2200 6240 50  0000 C CNN
+F 2 "handsolder:SOT-23-6handsoldering" H 2250 5650 50  0001 C CNN
+F 3 "http://www.ti.com/lit/ds/symlink/tpl5111.pdf" H 600 5800 50  0001 C CNN
+	1    2250 5650
+	1    0    0    -1
+$EndComp
 Text Label 2250 6050 3    50   ~ 0
 GND
@@
 Wire Wire Line
 	2650 4150 2700 4150
+Wire Wire Line
+	2750 5550 3050 5550
 Text Label 1650 5550 2    50   ~ 0
 GND
@@
 	2250 4150 2550 4150
 Wire Wire Line
-	4050 4700 4050 4400
+	2900 4400 2900 4100
 Wire Wire Line
 	2200 4150 2200 4350
@@
 L button-timer-v1.2.1_Coin_Cell-rescue:R-Device-button-timer-rescue-button-timer-v1.2-rescue-button-timer-v1.2-rescue R7
 U 1 1 602F7A06
-P 4500 5700
-F 0 "R7" H 4570 5746 50  0000 L CNN
-F 1 "10k" H 4570 5655 50  0000 L CNN
-F 2 "handsolder:R_0805_2012handsoldermod" V 4430 5700 50  0001 C CNN
-F 3 "~" H 4500 5700 50  0001 C CNN
-	1    4500 5700
-	-1   0    0    1
-$EndComp
+P 3200 5550
+F 0 "R7" H 3270 5596 50  0000 L CNN
+F 1 "10k" H 3270 5505 50  0000 L CNN
+F 2 "handsolder:R_0805_2012handsoldermod" V 3130 5550 50  0001 C CNN
+F 3 "~" H 3200 5550 50  0001 C CNN
+	1    3200 5550
+	0    -1   -1   0
+$EndComp
+Wire Wire Line
+	2700 4100 2900 4100
 Text Label 1500 5950 3    50   ~ 0
 GND
@@
 Wire Wire Line
 	1300 5650 1200 5650
-Connection ~ 4050 4400
-Wire Wire Line
-	5600 4600 5600 5850
-Wire Wire Line
-	4050 4400 4600 4400
-Wire Wire Line
-	4550 4950 5100 4950
-Wire Wire Line
-	4550 4950 4550 4700
-Wire Wire Line
-	4650 4500 4650 4600
-Wire Wire Line
-	4650 4600 4750 4600
-Connection ~ 5800 4750
-Wire Wire Line
-	5450 4750 5800 4750
-Wire Wire Line
-	5600 4600 5450 4600
+Connection ~ 2900 4100
+Wire Wire Line
+	4450 4300 4450 5550
+Wire Wire Line
+	2900 4100 3450 4100
+Wire Wire Line
+	3400 4650 3950 4650
+Wire Wire Line
+	3400 4650 3400 4400
+Wire Wire Line
+	3500 4200 3500 4300
+Wire Wire Line
+	3500 4300 3600 4300
+Connection ~ 4650 4450
+Wire Wire Line
+	4300 4450 4650 4450
+Wire Wire Line
+	4450 4300 4300 4300
 $Comp
 L button-timer-v1.2.1_Coin_Cell-rescue:TPS61097A-TPS-button-timer-v1.2-rescue U1
 U 1 1 6033543B
-P 5050 4450
-F 0 "U1" H 5100 4565 50  0000 C CNN
-F 1 "TPS61097A" H 5100 4474 50  0000 C CNN
-F 2 "handsolder:SOT-23-5_HandSolderingmod" H 5400 4400 50  0001 C CNN
-F 3 "" H 5400 4400 50  0001 C CNN
-	1    5050 4450
+P 3900 4150
+F 0 "U1" H 3950 4265 50  0000 C CNN
+F 1 "TPS61097A" H 3950 4174 50  0000 C CNN
+F 2 "handsolder:SOT-23-5_HandSolderingmod" H 4250 4100 50  0001 C CNN
+F 3 "" H 4250 4100 50  0001 C CNN
+	1    3900 4150
 	1    0    0    -1
 $EndComp
@@
 Text Label 6700 3600 0    50   ~ 0
 GPIO15
-Text Label 5850 4700 0    50   ~ 0
-VCC
-Text Label 5800 5050 0    50   ~ 0
-GND
-Wire Wire Line
-	5800 4750 5850 4750
+Text Label 4700 4400 0    50   ~ 0
+VCC
+Text Label 4650 4750 0    50   ~ 0
+GND
+Wire Wire Line
+	4650 4450 4700 4450
 $Comp
 L button-timer-v1.2.1_Coin_Cell-rescue:C-Device-button-timer-rescue-button-timer-v1.2-rescue-button-timer-v1.2-rescue C3
 U 1 1 602E3D4A
-P 5800 4900
-F 0 "C3" H 5915 4946 50  0000 L CNN
-F 1 "10uF" H 5915 4855 50  0000 L CNN
-F 2 "handsolder:C_0805_2012handsodermod" H 5838 4750 50  0001 C CNN
-F 3 "~" H 5800 4900 50  0001 C CNN
-	1    5800 4900
-	1    0    0    -1
-$EndComp
-Wire Wire Line
-	5850 4750 5850 4700
+P 4650 4600
+F 0 "C3" H 4765 4646 50  0000 L CNN
+F 1 "10uF" H 4765 4555 50  0000 L CNN
+F 2 "handsolder:C_0805_2012handsodermod" H 4688 4450 50  0001 C CNN
+F 3 "~" H 4650 4600 50  0001 C CNN
+	1    4650 4600
+	1    0    0    -1
+$EndComp
+Wire Wire Line
+	4700 4450 4700 4400
 $Comp
 L button-timer-v1.2.1_Coin_Cell-rescue:INDUCTOR-pspice-button-timer-rescue-button-timer-v1.2-rescue-button-timer-v1.2-rescue L1
 U 1 1 602E234D
-P 4300 4700
-F 0 "L1" H 4300 4915 50  0000 C CNN
-F 1 "4.7 uH" H 4300 4824 50  0000 C CNN
-F 2 "handsolder:SMD-1210_Pol_inductor" H 4300 4700 50  0001 C CNN
-F 3 "~" H 4300 4700 50  0001 C CNN
-	1    4300 4700
-	1    0    0    -1
-$EndComp
-Text Label 4750 4750 2    50   ~ 0
-GND
-Wire Wire Line
-	4600 4500 4650 4500
-Wire Wire Line
-	4600 4400 4600 4500
+P 3150 4400
+F 0 "L1" H 3150 4615 50  0000 C CNN
+F 1 "4.7 uH" H 3150 4524 50  0000 C CNN
+F 2 "handsolder:SMD-1210_Pol_inductor" H 3150 4400 50  0001 C CNN
+F 3 "~" H 3150 4400 50  0001 C CNN
+	1    3150 4400
+	1    0    0    -1
+$EndComp
+Text Label 3600 4450 2    50   ~ 0
+GND
+Wire Wire Line
+	3450 4200 3500 4200
+Wire Wire Line
+	3450 4100 3450 4200
 Text Label 6700 3100 0    50   ~ 0
 RX
@@
 $EndComp
 Wire Wire Line
-	4500 5850 5600 5850
+	3350 5550 4450 5550
 Wire Wire Line
 	2750 5650 3050 5650
@@
 Text Label 2850 4950 0    50   ~ 0
 GND
-$Comp
-L Timer:TPL5110 U2
-U 1 1 60350B91
-P 2250 5550
-F 0 "U2" H 2200 6131 50  0000 C CNN
-F 1 "TPL5110" H 2200 6040 50  0000 C CNN
-F 2 "Package_TO_SOT_SMD:SOT-23-6" H 2250 5550 50  0001 C CNN
-F 3 "http://www.ti.com/lit/ds/symlink/tpl5110.pdf" H 2050 5150 50  0001 C CNN
-	1    2250 5550
-	1    0    0    -1
-$EndComp
-Wire Wire Line
-	4500 5550 4500 4800
-Wire Wire Line
-	4500 4800 3950 4800
-Wire Wire Line
-	3950 4800 3950 4400
-Connection ~ 3950 4400
-Wire Wire Line
-	3950 4400 4050 4400
-Wire Wire Line
-	3350 5550 3350 4600
-Wire Wire Line
-	2750 5550 3350 5550
-$Comp
-L Transistor_FET:TSM2301ACX Q1
-U 1 1 6035BA2A
-P 3350 4400
-F 0 "Q1" V 3692 4400 50  0000 C CNN
-F 1 " TSM2323 " V 3601 4400 50  0000 C CNN
-F 2 "Package_TO_SOT_SMD:SOT-23" H 3550 4325 50  0001 L CIN
-F 3 "https://www.taiwansemi.com/products/datasheet/TSM2301A_C15.pdf" H 3350 4400 50  0001 L CNN
-	1    3350 4400
-	0    1    -1   0
-$EndComp
-Wire Wire Line
-	3550 4400 3550 4300
-Wire Wire Line
-	3550 4400 3950 4400
-Wire Wire Line
-	3150 4250 2750 4250
-Wire Wire Line
-	2750 4250 2750 4100
-Wire Wire Line
-	2750 4100 2700 4100
-Wire Wire Line
-	3150 4250 3150 4300
 $EndSCHEMATC

Commit message: 3D Models etwas verbessert
Parts:
- J1: footprint Connector_PinHeader_2.54mm:PinHeader_1x05_P2.54mm_Vertical -> handsolder:PinSocket_1x05_P2.54mm_Vertical_mod
- SW1: footprint Button_Switch_THT:SW_PUSH_6mm -> handsolder:SW_PUSH_6mm_H8mm_mod
- SW2: footprint Button_Switch_SMD:SW_SPST_EVQPE1 -> handsolder:SW_SPST_B3U-1000P_mod
Changed lines of the file:
@@
 F 0 "SW1" H 1200 5735 50  0000 C CNN
 F 1 "SW_Push" H 1200 5644 50  0000 C CNN
-F 2 "Button_Switch_THT:SW_PUSH_6mm" H 1200 5650 50  0001 C CNN
+F 2 "handsolder:SW_PUSH_6mm_H8mm_mod" H 1200 5650 50  0001 C CNN
 F 3 "~" H 1200 5650 50  0001 C CNN
 	1    1200 5450
@@
 F 0 "J1" H 8328 3576 50  0000 L CNN
 F 1 "Conn_01x05_Female" H 8328 3485 50  0000 L CNN
-F 2 "Connector_PinHeader_2.54mm:PinHeader_1x05_P2.54mm_Vertical" H 8300 3550 50  0001 C CNN
+F 2 "handsolder:PinSocket_1x05_P2.54mm_Vertical_mod" H 8300 3550 50  0001 C CNN
 F 3 "~" H 8300 3550 50  0001 C CNN
 	1    8300 3550
@@
 F 0 "SW2" H 7800 2335 50  0000 C CNN
 F 1 "SW_Push" H 7800 2244 50  0000 C CNN
-F 2 "Button_Switch_SMD:SW_SPST_EVQPE1" H 7800 2250 50  0001 C CNN
+F 2 "handsolder:SW_SPST_B3U-1000P_mod" H 7800 2250 50  0001 C CNN
 F 3 "~" H 7800 2250 50  0001 C CNN
 	1    7800 2050
