File: button_timer_v1.2_mosfet[EXPERIMENT]/button_timer_v1.2_mosfet.sch (KiCad schematic (older format))
At the start: 29 parts, among them J1 Conn_01x05_Female, Q1 TSM2301ACX, SW1 SW_Push, SW2 SW_Push, U1 TPS61097A, U2 AP2112K-3.3, U3 TPL5111, X1 ESP-12E

Commit message: 23.02 13:31
Parts:
- added C5: 100nF, handsolder:C_0805_2012handsodermod, symbol Device:C
Connections:
- net GND: now also C5.2
- net at BT1.1 (+), BT2.1 (+), C1.2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: now also C5.1
Changed lines of the file:
@@
 GND
 Wire Wire Line
-	2550 4150 2550 5050
+	2550 4150 2550 4900
 Wire Wire Line
 	2550 5050 2250 5050
@@
 Text Label 2800 6550 0    50   ~ 0
 GND
+$Comp
+L Device:C C5
+U 1 1 60350256
+P 2400 4900
+F 0 "C5" V 2148 4900 50  0000 C CNN
+F 1 "100nF" V 2239 4900 50  0000 C CNN
+F 2 "handsolder:C_0805_2012handsodermod" H 2438 4750 50  0001 C CNN
+F 3 "~" H 2400 4900 50  0001 C CNN
+	1    2400 4900
+	0    1    1    0
+$EndComp
+Connection ~ 2550 4900
+Wire Wire Line
+	2550 4900 2550 5050
+Text Label 2250 4900 2    50   ~ 0
+GND
 $EndSCHEMATC

Commit message: 3D Models etwas verbessert
Parts:
- C5: footprint handsolder:C_0805_2012handsodermod -> Capacitor_SMD:C_0805_2012Metric_Pad1.18x1.45mm_HandSolder
- J1: footprint Connector_PinHeader_2.54mm:PinHeader_1x05_P2.54mm_Vertical -> handsolder:PinSocket_1x05_P2.54mm_Vertical_mod
- SW1: footprint Button_Switch_THT:SW_PUSH_6mm -> handsolder:SW_PUSH_6mm_H8mm_mod
- SW2: footprint Button_Switch_SMD:SW_SPST_EVQPE1 -> handsolder:SW_SPST_B3U-1000P_mod
Changed lines of the file:
@@
 F 0 "SW2" H 7800 2335 50  0000 C CNN
 F 1 "SW_Push" H 7800 2244 50  0000 C CNN
-F 2 "Button_Switch_SMD:SW_SPST_EVQPE1" H 7800 2250 50  0001 C CNN
+F 2 "handsolder:SW_SPST_B3U-1000P_mod" H 7800 2250 50  0001 C CNN
 F 3 "~" H 7800 2250 50  0001 C CNN
 	1    7800 2050
@@
 F 0 "SW1" H 1100 5935 50  0000 C CNN
 F 1 "SW_Push" H 1100 5844 50  0000 C CNN
-F 2 "Button_Switch_THT:SW_PUSH_6mm" H 1100 5850 50  0001 C CNN
+F 2 "handsolder:SW_PUSH_6mm_H8mm_mod" H 1100 5850 50  0001 C CNN
 F 3 "~" H 1100 5850 50  0001 C CNN
 	1    1100 5650
@@
 F 0 "J1" H 8328 3576 50  0000 L CNN
 F 1 "Conn_01x05_Female" H 8328 3485 50  0000 L CNN
-F 2 "Connector_PinHeader_2.54mm:PinHeader_1x05_P2.54mm_Vertical" H 8300 3550 50  0001 C CNN
+F 2 "handsolder:PinSocket_1x05_P2.54mm_Vertical_mod" H 8300 3550 50  0001 C CNN
 F 3 "~" H 8300 3550 50  0001 C CNN
 	1    8300 3550
@@
 F 0 "C5" V 2148 4900 50  0000 C CNN
 F 1 "100nF" V 2239 4900 50  0000 C CNN
-F 2 "handsolder:C_0805_2012handsodermod" H 2438 4750 50  0001 C CNN
+F 2 "Capacitor_SMD:C_0805_2012Metric_Pad1.18x1.45mm_HandSolder" H 2438 4750 50  0001 C CNN
 F 3 "~" H 2400 4900 50  0001 C CNN
 	1    2400 4900
