File: button timer v1.2.3_Coin_Cell[TPL5111]/button timer v1.2.3_Coin_Cell[TPL5111].sch (KiCad schematic (older format))
At the start: 25 parts, among them J1 Conn_01x05_Female, Q1 IRF540N, SW1 SW_Push, SW2 SW_Push, U1 TPS61097A, U3 TPL5111, X1 ESP-12E

Commit message: :rocket: :moon: :100:
Other:
- note added: "ANGUCKEN!!!"
Changed lines of the file:
@@
 Text Label 6000 5750 0    50   ~ 0
 GND_ESP
+Text Notes 5000 5350 0    50   ~ 0
+ANGUCKEN!!!
 $EndSCHEMATC
