File: button timer v1.2.3_[Coin_Cell&LIPO][TPL5111]/button timer v1.2.3_[Coin_Cell&LIPO][TPL5111].kicad_pcb (KiCad board)
At the start: 2 copper layers, 21 x 51.6 mm, 29 parts, among them J1 Conn_01x05_Female, Q1 mmbt222, SW1 SW_Push, SW2 SW_Push, U1 TPS61097A, U2 AP2112K-3.3, U3 TPL5111, X1 ESP-12E

Commit message: :rocket: :moon: :100:
Routing:
- net Net-(BT1-Pad1): track 47.1 -> 46.1 mm
Other:
- board text removed: "JP1 = Coin Cell JP2 = LIPO"
