File: button_timer_v1.2.3_lipo[TPL5110] -- UNNESSARY/button_timer_v1.2.3_lipo[TPL5110].sch (KiCad schematic (older format))
At the start: 25 parts, among them J1 Conn_01x05_Female, Q1 TSM2301ACX, Q2 TSM2301ACX, SW1 SW_Push, SW2 SW_Push, U1 TPL5110, U2 AP2112K-3.3, X1 ESP-12E

Commit message: cap between esp vcc and ground added
Parts:
- added C6: TAJB476M010TNJ, CAPPM3528X210N, symbol SamacSys_Parts:TAJB476M010TNJ
Connections:
- net GND: now also C6.2
- net VCC_ESP: now also C6.1
Changed lines of the file:
@@
 Text Label 4750 5600 0    50   ~ 0
 VCC_ESP
+$Comp
+L SamacSys_Parts:TAJB476M010TNJ C6
+U 1 1 60363F81
+P 5300 3700
+F 0 "C6" V 5504 3830 50  0000 L CNN
+F 1 "TAJB476M010TNJ" V 5595 3830 50  0000 L CNN
+F 2 "CAPPM3528X210N" H 5650 3750 50  0001 L CNN
+F 3 "http://datasheets.avx.com/TAJ.pdf" H 5650 3650 50  0001 L CNN
+F 4 "Tantalum Capacitors - Solid SMD 10volts 47uF 20%" H 5650 3550 50  0001 L CNN "Description"
+F 5 "2.1" H 5650 3450 50  0001 L CNN "Height"
+F 6 "AVX" H 5650 3350 50  0001 L CNN "Manufacturer_Name"
+F 7 "TAJB476M010TNJ" H 5650 3250 50  0001 L CNN "Manufacturer_Part_Number"
+F 8 "581-TAJB476M010TNJ" H 5650 3150 50  0001 L CNN "Mouser Part Number"
+F 9 "https://www.mouser.co.uk/ProductDetail/AVX/TAJB476M010TNJ?qs=pYVYkI7xuRVorIKKgcxm0A%3D%3D" H 5650 3050 50  0001 L CNN "Mouser Price/Stock"
+F 10 "TAJB476M010TNJ" H 5650 2950 50  0001 L CNN "Arrow Part Number"
+F 11 "https://www.arrow.com/en/products/tajb476m010tnj/avx" H 5650 2850 50  0001 L CNN "Arrow Price/Stock"
+	1    5300 3700
+	0    1    1    0
+$EndComp
+Text Label 5300 4200 3    50   ~ 0
+GND
 $EndSCHEMATC
