File: button_timer v1.2.3_Coin_Cell[TPL5111]/_autosave-button timer v1.2.3_Coin_Cell[TPL5111].sch (KiCad schematic (older format))
At the start: 26 parts, among them J1 Conn_01x05_Female, Q1 TSM2323, Q2 TSM2323, SW1 SW_Push, SW2 SW_Push, U1 TPS61097A, U2 TPL5110, X1 ESP-12E

Commit message: Added 100nF decoupling capacitors between VCC and Ground of the ESP
Parts:
- removed Q1, Q2: TSM2323, Package_TO_SOT_SMD:SOT-23, symbol Transistor_FET:TSM2301ACX
- removed R1: 10k, handsolder:R_0805_2012handsoldermod, symbol button_timer-v1.2.3_Coin_Cell[TPL5110]-rescue:R-Device-button-timer-rescue-butt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
- removed U2: TPL5110, Package_TO_SOT_SMD:SOT-23-6, symbol Timer:TPL5110
- added C6: TAJB476M010TNJ, CAPPM3528X210N, symbol SamacSys_Parts:TAJB476M010TNJ
- added C7: 100nF, handsolder:C_0402_1005Metric_Pad0.74x0.62mm_HandSoldermod, symbol Device:C
- added Q1: mmbt2222, Package_TO_SOT_SMD:SOT-23, symbol Transistor_FET:IRF540N
- added R10: 10k, Resistor_SMD:R_0603_1608Metric_Pad0.98x0.95mm_HandSolder, symbol Device:R
- added U3: TPL5111, handsolder:SOT-23-6handsoldering, symbol button-timer-v1.2.3_Coin_Cell[TPL5111]-rescue:TPL5111-Timer-button-timer-rescue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
- BT1: symbol button_timer-v1.2.3_Coin_Cell[TPL5110]-rescue:Battery_Cell-Device-button-timer-rescue-button-timer-v1.2-rescue-button-t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 -> button-timer-v1.2.3_Coin_Cell[TPL5111]-rescue:Battery_Cell-Device-button-timer-rescue-button-timer-v1.2-rescue-button-t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
- C1, C2, C3: symbol button_timer-v1.2.3_Coin_Cell[TPL5110]-rescue:C-Device-button-timer-rescue-button-timer-v1.2-rescue-button-timer-v1.2-r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 -> button-timer-v1.2.3_Coin_Cell[TPL5111]-rescue:C-Device-button-timer-rescue-button-timer-v1.2-rescue-button-timer-v1.2-r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
- D1, D2: symbol button_timer-v1.2.3_Coin_Cell[TPL5110]-rescue:LED-Device-button-timer-rescue-button-timer-v1.2-rescue-button-timer-v1.2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 -> button-timer-v1.2.3_Coin_Cell[TPL5111]-rescue:LED-Device-button-timer-rescue-button-timer-v1.2-rescue-button-timer-v1.2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
- J1: symbol button_timer-v1.2.3_Coin_Cell[TPL5110]-rescue:Conn_01x05_Female-Connector-button-timer-rescue-button-timer-v1.2-rescue-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 -> button-timer-v1.2.3_Coin_Cell[TPL5111]-rescue:Conn_01x05_Female-Connector-button-timer-rescue-button-timer-v1.2-rescue-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
- L1: symbol button_timer-v1.2.3_Coin_Cell[TPL5110]-rescue:INDUCTOR-pspice-button-timer-rescue-button-timer-v1.2-rescue-button-timer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 -> button-timer-v1.2.3_Coin_Cell[TPL5111]-rescue:INDUCTOR-pspice-button-timer-rescue-button-timer-v1.2-rescue-button-timer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
- R2, R3, R4, R5, R6, R7, R8, R9: symbol button_timer-v1.2.3_Coin_Cell[TPL5110]-rescue:R-Device-button-timer-rescue-button-timer-v1.2-rescue-button-timer-v1.2-r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 -> button-timer-v1.2.3_Coin_Cell[TPL5111]-rescue:R-Device-button-timer-rescue-button-timer-v1.2-rescue-button-timer-v1.2-r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
- SW1, SW2: symbol button_timer-v1.2.3_Coin_Cell[TPL5110]-rescue:SW_Push-Switch-button-timer-rescue-button-timer-v1.2-rescue-button-timer-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 -> button-timer-v1.2.3_Coin_Cell[TPL5111]-rescue:SW_Push-Switch-button-timer-rescue-button-timer-v1.2-rescue-button-timer-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
- U1: symbol button_timer-v1.2.3_Coin_Cell[TPL5110]-rescue:TPS61097A-TPS-button-timer-v1.2-rescue-button-timer-v1.2.1_Coin_Cell-resc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 -> button-timer-v1.2.3_Coin_Cell[TPL5111]-rescue:TPS61097A-TPS-button-timer-v1.2-rescue-button-timer-v1.2.1_Coin_Cell-resc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
- X1: symbol button_timer-v1.2.3_Coin_Cell[TPL5110]-rescue:ESP-12E-ardafruit-button-timer-rescue-button-timer-v1.2-rescue-button-tim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 -> button-timer-v1.2.3_Coin_Cell[TPL5111]-rescue:ESP-12E-ardafruit-button-timer-rescue-button-timer-v1.2-rescue-button-tim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
Connections:
- net labels added: GND_ESP
- net labels removed: ESP_VCC
- wire segments 54 -> 46
Other:
- moved on the sheet: C3, L1, R7, U1
