File: button_timer v1.2_[Coin_Cell&LIPO][NO TIMER]/button timer v1.2_[Coin_Cell&LIPO][NO TIMER].sch (KiCad schematic (older format))
At the start: 22 parts, among them J1 Conn_01x05_Female, SW1 SW_Push, SW2 SW_Push, U1 TPS61097A, U2 AP2112K-3.3, X1 ESP-12E

Commit message: cap between esp vcc and ground added
Parts:
- added C4: TAJB476M010TNJ, CAPPM3528X210N, symbol SamacSys_Parts:TAJB476M010TNJ
Connections:
- net GND: now also C4.2
- net VCC: now also C4.1
Changed lines of the file:
@@
 Wire Wire Line
 	3300 5100 3300 5650
+$Comp
+L SamacSys_Parts:TAJB476M010TNJ C4
+U 1 1 603640CA
+P 5300 3700
+F 0 "C4" V 5504 3830 50  0000 L CNN
+F 1 "TAJB476M010TNJ" V 5595 3830 50  0000 L CNN
+F 2 "CAPPM3528X210N" H 5650 3750 50  0001 L CNN
+F 3 "http://datasheets.avx.com/TAJ.pdf" H 5650 3650 50  0001 L CNN
+F 4 "Tantalum Capacitors - Solid SMD 10volts 47uF 20%" H 5650 3550 50  0001 L CNN "Description"
+F 5 "2.1" H 5650 3450 50  0001 L CNN "Height"
+F 6 "AVX" H 5650 3350 50  0001 L CNN "Manufacturer_Name"
+F 7 "TAJB476M010TNJ" H 5650 3250 50  0001 L CNN "Manufacturer_Part_Number"
+F 8 "581-TAJB476M010TNJ" H 5650 3150 50  0001 L CNN "Mouser Part Number"
+F 9 "https://www.mouser.co.uk/ProductDetail/AVX/TAJB476M010TNJ?qs=pYVYkI7xuRVorIKKgcxm0A%3D%3D" H 5650 3050 50  0001 L CNN "Mouser Price/Stock"
+F 10 "TAJB476M010TNJ" H 5650 2950 50  0001 L CNN "Arrow Part Number"
+F 11 "https://www.arrow.com/en/products/tajb476m010tnj/avx" H 5650 2850 50  0001 L CNN "Arrow Price/Stock"
+	1    5300 3700
+	0    1    1    0
+$EndComp
+Text Label 5300 4200 0    50   ~ 0
+GND
 $EndSCHEMATC

Commit message: Added 100nF decoupling capacitors between VCC and Ground of the ESP
Parts:
- added C?: 100nF, handsolder:C_0402_1005Metric_Pad0.74x0.62mm_HandSoldermod, symbol Device:C
Connections:
- net GND: now also C?.2
- net VCC: now also C?.1
Changed lines of the file:
@@
 Text Label 5300 4200 0    50   ~ 0
 GND
+$Comp
+L Device:C C?
+U 1 1 60368135
+P 5000 3900
+F 0 "C?" H 5115 3946 50  0000 L CNN
+F 1 "100nF" H 5115 3855 50  0000 L CNN
+F 2 "handsolder:C_0402_1005Metric_Pad0.74x0.62mm_HandSoldermod" H 5038 3750 50  0001 C CNN
+F 3 "~" H 5000 3900 50  0001 C CNN
+	1    5000 3900
+	1    0    0    -1
+$EndComp
+Wire Wire Line
+	5000 3750 5000 3700
+Wire Wire Line
+	5000 3700 5300 3700
+Connection ~ 5300 3700
+Wire Wire Line
+	5000 4050 5000 4200
+Wire Wire Line
+	5000 4200 5300 4200
 $EndSCHEMATC
