File: button_timer v1.2_[Coin_Cell&LIPO][TPL5110]/_autosave-button timer v1.2_[Coin_Cell&LIPO][TPL5110].sch (KiCad schematic (older format))
At the start: 30 parts, among them J1 Conn_01x05_Female, Q1 mmbt222, SW1 SW_Push, SW2 SW_Push, U1 TPS61097A, U2 AP2112K-3.3, U3 TPL5111, X1 ESP-12E

Commit message: Added 100nF decoupling capacitors between VCC and Ground of the ESP
Parts:
- removed JP1: Jumper Coin Cell, Jumper:SolderJumper-2_P1.3mm_Open_RoundedPad1.0x1.5mm, symbol button-timer-v1.2.3_[Coin_Cell&LIPO][TPL5111]-rescue:Jumper_NO_Small-Device-but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
- removed JP2: Jumper LIPO, Jumper:SolderJumper-2_P1.3mm_Open_RoundedPad1.0x1.5mm, symbol button-timer-v1.2.3_[Coin_Cell&LIPO][TPL5111]-rescue:Jumper_NO_Small-Device-but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
- removed Q1: mmbt222, Package_TO_SOT_SMD:SOT-23, symbol Transistor_FET:IRF540N
- removed R1: 10k, handsolder:R_0603_1608Metric_Pad0.98x0.95mm_HandSolder_mod, symbol Device:R
- removed U3: TPL5111, handsolder:SOT-23-6handsoldering, symbol button-timer-v1.2.3_[Coin_Cell&LIPO][TPL5111]-rescue:TPL5111-Timer-button-timer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
- added C7: 100nF, handsolder:C_0402_1005Metric_Pad0.74x0.62mm_HandSoldermod, symbol Device:C
- added Q1: TSM2301ACX, Package_TO_SOT_SMD:SOT-23, symbol Transistor_FET:TSM2301ACX
- added R1: 10k, handsolder:R_0805_2012handsoldermod, symbol button-timer-v1.2-rescue:R-Device-button-timer-rescue-button-timer-v1.2-rescue-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
- added U3: TPL5110, handsolder:SOT-23-6handsoldering, symbol Timer:TPL5110
- BT1, BT2: symbol button-timer-v1.2.3_[Coin_Cell&LIPO][TPL5111]-rescue:Battery_Cell-Device-button-timer-rescue-button-timer-v1.2-rescue-b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 -> button-timer-v1.2-rescue:Battery_Cell-Device-button-timer-rescue-button-timer-v1.2-rescue-button-timer-v1.2-rescue-butt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
- C1, C2, C3: symbol button-timer-v1.2.3_[Coin_Cell&LIPO][TPL5111]-rescue:C-Device-button-timer-rescue-button-timer-v1.2-rescue-button-timer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 -> button-timer-v1.2-rescue:C-Device-button-timer-rescue-button-timer-v1.2-rescue-button-timer-v1.2-rescue-button-timer-v1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
- D1, D2: symbol button-timer-v1.2.3_[Coin_Cell&LIPO][TPL5111]-rescue:LED-Device-button-timer-rescue-button-timer-v1.2-rescue-button-tim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 -> button-timer-v1.2-rescue:LED-Device-button-timer-rescue-button-timer-v1.2-rescue-button-timer-v1.2-rescue-button-timer-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
- J1: symbol button-timer-v1.2.3_[Coin_Cell&LIPO][TPL5111]-rescue:Conn_01x05_Female-Connector-button-timer-rescue-button-timer-v1.2-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 -> button-timer-v1.2-rescue:Conn_01x05_Female-Connector-button-timer-rescue-button-timer-v1.2-rescue-button-timer-v1.2-res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
- L1: symbol button-timer-v1.2.3_[Coin_Cell&LIPO][TPL5111]-rescue:INDUCTOR-pspice-button-timer-rescue-button-timer-v1.2-rescue-butto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 -> button-timer-v1.2-rescue:INDUCTOR-pspice-button-timer-rescue-button-timer-v1.2-rescue-button-timer-v1.2-rescue-button-t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
- R2, R3, R4, R5, R6, R7, R8, R9: symbol button-timer-v1.2.3_[Coin_Cell&LIPO][TPL5111]-rescue:R-Device-button-timer-rescue-button-timer-v1.2-rescue-button-timer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 -> button-timer-v1.2-rescue:R-Device-button-timer-rescue-button-timer-v1.2-rescue-button-timer-v1.2-rescue-button-timer-v1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
- SW1, SW2: symbol button-timer-v1.2.3_[Coin_Cell&LIPO][TPL5111]-rescue:SW_Push-Switch-button-timer-rescue-button-timer-v1.2-rescue-button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 -> button-timer-v1.2-rescue:SW_Push-Switch-button-timer-rescue-button-timer-v1.2-rescue-button-timer-v1.2-rescue-button-ti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
- U1: symbol button-timer-v1.2.3_[Coin_Cell&LIPO][TPL5111]-rescue:TPS61097A-TPS-button-timer-v1.2-rescue-button-timer-v1.2-rescue-bu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 -> button-timer-v1.2-rescue:TPS61097A-TPS-button-timer-v1.2-rescue-button-timer-v1.2-rescue
- U2: symbol button-timer-v1.2.3_[Coin_Cell&LIPO][TPL5111]-rescue:AP2112K-3.3-Regulator_Linear-button-timer-rescue-button-timer-v1.2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 -> button-timer-v1.2-rescue:AP2112K-3.3-Regulator_Linear-button-timer-rescue-button-timer-v1.2-rescue-button-timer-v1.2-re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
- X1: symbol button-timer-v1.2.3_[Coin_Cell&LIPO][TPL5111]-rescue:ESP-12E-ardafruit-button-timer-rescue-button-timer-v1.2-rescue-but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 -> button-timer-v1.2-rescue:ESP-12E-ardafruit-button-timer-rescue-button-timer-v1.2-rescue-button-timer-v1.2-rescue-button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
Connections:
- net labels removed: GND_ESP
- wire segments 60 -> 66
