File: button_timer_v1.2.3_lipo[TPL5110] -- unnecessary/button_timer_v1.2.3_lipo[TPL5110].sch (KiCad schematic (older format))
At the start: 26 parts, among them J1 Conn_01x05_Female, Q1 TSM2301ACX, SW1 SW_Push, SW2 SW_Push, U1 TPL5110, U2 AP2112K-3.3, X1 ESP-12E

Commit message: Added 100nF decoupling capacitors between VCC and Ground of the ESP
Parts:
- removed C6: 47uF, SamacSys_Parts:CAPPM3528X210N, symbol Device:CP
- removed C?: 100nF, handsolder:C_0402_1005Metric_Pad0.74x0.62mm_HandSoldermod, symbol Device:C
- added C6: TAJB476M010TNJ, CAPPM3528X210N, symbol SamacSys_Parts:TAJB476M010TNJ
- added C?: 100nF, handsolder:C_0402_1005Metric_Pad0.74x0.62mm_HandSoldermod, symbol Device:C
- added Q2: TSM2301ACX, Package_TO_SOT_SMD:SOT-23, symbol Transistor_FET:TSM2301ACX
Connections:
- net labels added: VCC_ESP
- wire segments 36 -> 40
Changed lines of the file:
@@
 GND
 Text Label 5300 3700 2    50   ~ 0
-VCC
+VCC_ESP
 Text Label 7900 3250 2    50   ~ 0
 VCC
@@
 DRV is low when ACTIVE! [ONLY TPL5110]
 $Comp
-L Device:CP C6
-U 1 1 60362D5E
-P 5300 3850
-F 0 "C6" H 5418 3896 50  0000 L CNN
-F 1 "47uF" H 5418 3805 50  0000 L CNN
-F 2 "SamacSys_Parts:CAPPM3528X210N" H 5338 3700 50  0001 C CNN
-F 3 "~" H 5300 3850 50  0001 C CNN
-	1    5300 3850
-	1    0    0    -1
-$EndComp
-Text Label 5300 4000 3    50   ~ 0
+L Transistor_FET:TSM2301ACX Q2
+U 1 1 60357B62
+P 4550 5700
+F 0 "Q2" V 4892 5700 50  0000 C CNN
+F 1 "TSM2301ACX" V 4801 5700 50  0000 C CNN
+F 2 "Package_TO_SOT_SMD:SOT-23" H 4750 5625 50  0001 L CIN
+F 3 "https://www.taiwansemi.com/products/datasheet/TSM2301A_C15.pdf" H 4550 5700 50  0001 L CNN
+	1    4550 5700
+	0    1    -1   0
+$EndComp
+Wire Wire Line
+	3800 5250 3800 5900
+Wire Wire Line
+	3800 5900 4550 5900
+Connection ~ 3800 5250
+Text Label 4350 5600 2    50   ~ 0
+VCC
+Text Label 4750 5600 0    50   ~ 0
+VCC_ESP
+$Comp
+L SamacSys_Parts:TAJB476M010TNJ C6
+U 1 1 60363F81
+P 5300 3700
+F 0 "C6" V 5504 3830 50  0000 L CNN
+F 1 "TAJB476M010TNJ" V 5595 3830 50  0000 L CNN
+F 2 "CAPPM3528X210N" H 5650 3750 50  0001 L CNN
+F 3 "http://datasheets.avx.com/TAJ.pdf" H 5650 3650 50  0001 L CNN
+F 4 "Tantalum Capacitors - Solid SMD 10volts 47uF 20%" H 5650 3550 50  0001 L CNN "Description"
+F 5 "2.1" H 5650 3450 50  0001 L CNN "Height"
+F 6 "AVX" H 5650 3350 50  0001 L CNN "Manufacturer_Name"
+F 7 "TAJB476M010TNJ" H 5650 3250 50  0001 L CNN "Manufacturer_Part_Number"
+F 8 "581-TAJB476M010TNJ" H 5650 3150 50  0001 L CNN "Mouser Part Number"
+F 9 "https://www.mouser.co.uk/ProductDetail/AVX/TAJB476M010TNJ?qs=pYVYkI7xuRVorIKKgcxm0A%3D%3D" H 5650 3050 50  0001 L CNN "Mouser Price/Stock"
+F 10 "TAJB476M010TNJ" H 5650 2950 50  0001 L CNN "Arrow Part Number"
+F 11 "https://www.arrow.com/en/products/tajb476m010tnj/avx" H 5650 2850 50  0001 L CNN "Arrow Price/Stock"
+	1    5300 3700
+	0    1    1    0
+$EndComp
+Text Label 5300 4200 3    50   ~ 0
 GND
 $Comp
 L Device:C C?
-U 1 1 60367D4C
+U 1 1 60367E56
 P 5000 3850
 F 0 "C?" H 5115 3896 50  0000 L CNN
@@
 Connection ~ 5300 3700
 Wire Wire Line
-	5000 4000 5300 4000
+	5000 4000 5200 4000
+Wire Wire Line
+	5200 4000 5200 4200
+Wire Wire Line
+	5200 4200 5300 4200
 $EndSCHEMATC
