File: button_timer_v1.2.3_lipo[TPL5110] -- unnecessary/button_timer_v1.2.3_lipo[TPL5110].kicad_pcb (KiCad board)
At the start: 2 copper layers, 21 x 41.7 mm, 26 parts, among them J1 Conn_01x05_Female, Q1 TSM2301ACX, SW1 SW_Push, SW2 SW_Push, U1 TPL5110, U2 AP2112K-3.3, X1 ESP-12E

Commit message: Added 100nF decoupling capacitors between VCC and Ground of the ESP
Parts:
- added Q2: TSM2301ACX, handsolder:SOT-23, B.Cu at (129.5, 87.6)
- C6: value 47uF -> TAJB476M010TNJ
- C7: moved to F.Cu
- moved C6 4.87 mm to (133.4, 81.5), turned to 270 degrees
- moved C7 4.04 mm to (134.7, 78.3), turned to 0 degrees
- moved C3 3.02 mm to (121.0, 83.1)
- moved U2 3.02 mm to (125.3, 83.1)
- moved R7 3.02 mm to (129.8, 82.9)
Connections:
- C6 pad 1: /VCC -> /VCC_ESP
- C7 pad 1: /VCC -> /VCC_ESP
- X1 pad 8: /VCC -> /VCC_ESP
Routing:
- net Net-(Q1-Pad1): track 1.98 -> 20.9 mm
- net /VCC_ESP: track 0.00 -> 12.9 mm, vias 0 -> 1
- net /GND: track 92.4 -> 104.0 mm
- net Net-(Q1-Pad3): track 18.9 -> 13.0 mm
- net /VCC: track 46.5 -> 43.7 mm, vias 2 -> 1
- net /EN: track 15.7 -> 16.9 mm, vias 2 -> 0
Other:
- board text added: "Button - LIPO v.1.2.3 TIMER 5110"
- board text added: "V1.2.3 ONLY LIPO TIMER TPL5110"
- board text removed: "Button - LIPO v.1.2.1 TIMER 5110"
- board text removed: "V1.2.1 ONLY LIPO TIMER TPL5110"
