File: button_timer_v1.2.3_lipo[TPL5111] -- unnecessary/_autosave-button_timer_v1.2.3_lipo[TPL5111].sch (KiCad schematic (older format))
At the start: 26 parts, among them J1 Conn_01x05_Female, Q1 TSM2301ACX, Q2 TSM2301ACX, SW1 SW_Push, SW2 SW_Push, U1 TPL5110, U2 AP2112K-3.3, X1 ESP-12E

Commit message: Added 100nF decoupling capacitors between VCC and Ground of the ESP
Parts:
- removed C?: TAJB476M010TNJ, CAPPM3528X210N, symbol SamacSys_Parts:TAJB476M010TNJ
- removed Q1, Q2: TSM2301ACX, Package_TO_SOT_SMD:SOT-23, symbol Transistor_FET:TSM2301ACX
- removed R1: 10k, handsolder:R_0805_2012handsoldermod, symbol button-timer-v1.2-rescue:R-Device-button-timer-rescue-button-timer-v1.2-rescue-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
- removed R7: 100k, handsolder:R_0805_2012handsoldermod, symbol Device:R
- removed U1: TPL5110, handsolder:SOT-23-6handsoldering, symbol Timer:TPL5110
- added C6: TAJB476M010TNJ, CAPPM3528X210N, symbol SamacSys_Parts:TAJB476M010TNJ
- added C7: 100nF, handsolder:C_0402_1005Metric_Pad0.74x0.62mm_HandSoldermod, symbol Device:C
- added Q1: mmbt2222, Package_TO_SOT_SMD:SOT-23, symbol Transistor_FET:IRF540N
- added R1: 10k, handsolder:R_0603_1608Metric_Pad0.98x0.95mm_HandSolder_mod, symbol Device:R
- added R7: 10k, handsolder:R_0805_2012handsoldermod, symbol button-timer-v1.2-rescue:R-Device-button-timer-rescue-button-timer-v1.2-rescue-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
- added U3: TPL5111, handsolder:SOT-23-6handsoldering, symbol button-timer-v1.2-rescue:TPL5111-Timer-button-timer-rescue-button-timer-v1.2-re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
- C5: footprint handsolder:C_0805_2012handsodermod -> handsolder:C_0402_1005Metric_Pad0.74x0.62mm_HandSoldermod
- J1: footprint handsolder:PinSocket_1x05_P2.54mm_Vertical_mod -> Connector_PinSocket_2.54mm:PinSocket_1x05_P2.54mm_Vertical
- SW1: footprint handsolder:SW_PUSH_6mm_H8mm_mod -> Button_Switch_THT:SW_PUSH_6mm_H8mm
- SW2: footprint handsolder:SW_SPST_B3U-1000P_mod -> Button_Switch_SMD:SW_SPST_B3U-1000P
Connections:
- net labels added: GND_ESP
- net labels removed: VCC_ESP
- wire segments 36 -> 40
Other:
- note removed: "DRV is low when ACTIVE! [ONLY TPL5110]"
- moved on the sheet: BT1, C1, C3, C4, D1, R6, R8, SW1, U2
