File: button_v1.2.2_lipo[NO TIMER]/button_v1.2.2_lipo.sch (KiCad schematic (older format))
At the start: 17 parts, among them J1 Conn_01x05_Female, SW1 SW_Push, SW2 SW_Push, U2 AP2112K-3.3, X1 ESP-12E

Commit message: :airplane:
Connections:
- net GND: no longer D1.1 (K)
- net RST: now also R6.2, SW1.1
- net VCC: now also D1.1 (K)
Changed lines of the file:
@@
 	3350 2300 3350 2600
 Text Label 3350 2600 3    50   ~ 0
-GND
+VCC
 Wire Wire Line
 	2200 4150 2200 4350
@@
 Text Label 4750 2500 0    50   ~ 0
 GND
+Wire Wire Line
+	4050 2500 4050 2700
+Wire Wire Line
+	4050 2700 3950 2700
+Connection ~ 4050 2500
+Text Label 3950 2700 2    50   ~ 0
+RST
 $EndSCHEMATC

Commit message: :rocket: :full_moon_with_face:
Connections:
- net VCC: now also D1.2 (A); no longer D1.1 (K)
- net at R6.1: now also D1.1 (K); no longer D1.2 (A)
Other:
- moved on the sheet: D1
Changed lines of the file:
@@
 F 3 "~" H 3600 2300 50  0001 C CNN
 	1    3600 2300
-	1    0    0    -1
+	-1   0    0    1
 $EndComp
 Wire Wire Line

Commit message: 3D Models etwas verbessert
Parts:
- J1: footprint Connector_PinHeader_2.54mm:PinHeader_1x05_P2.54mm_Vertical -> handsolder:PinSocket_1x05_P2.54mm_Vertical_mod
- SW1: footprint Button_Switch_THT:SW_PUSH_6mm -> handsolder:SW_PUSH_6mm_H8mm_mod
- SW2: footprint Button_Switch_SMD:SW_SPST_EVQPE1 -> handsolder:SW_SPST_B3U-1000P_mod
Changed lines of the file:
@@
 F 0 "SW2" H 8000 3385 50  0000 C CNN
 F 1 "SW_Push" H 8000 3294 50  0000 C CNN
-F 2 "Button_Switch_SMD:SW_SPST_EVQPE1" H 8000 3300 50  0001 C CNN
+F 2 "handsolder:SW_SPST_B3U-1000P_mod" H 8000 3300 50  0001 C CNN
 F 3 "~" H 8000 3300 50  0001 C CNN
 	1    8000 3100
@@
 F 0 "SW1" H 4250 2785 50  0000 C CNN
 F 1 "SW_Push" H 4250 2694 50  0000 C CNN
-F 2 "Button_Switch_THT:SW_PUSH_6mm" H 4250 2700 50  0001 C CNN
+F 2 "handsolder:SW_PUSH_6mm_H8mm_mod" H 4250 2700 50  0001 C CNN
 F 3 "~" H 4250 2700 50  0001 C CNN
 	1    4250 2500
@@
 F 0 "J1" H 8128 3476 50  0000 L CNN
 F 1 "Conn_01x05_Female" H 8128 3385 50  0000 L CNN
-F 2 "Connector_PinHeader_2.54mm:PinHeader_1x05_P2.54mm_Vertical" H 8100 3450 50  0001 C CNN
+F 2 "handsolder:PinSocket_1x05_P2.54mm_Vertical_mod" H 8100 3450 50  0001 C CNN
 F 3 "~" H 8100 3450 50  0001 C CNN
 	1    8100 3450

Commit message: cap between esp vcc and ground added
Parts:
- added C4: TAJB476M010TNJ, CAPPM3528X210N, symbol SamacSys_Parts:TAJB476M010TNJ
Connections:
- net GND: now also C4.2
- net VCC: now also C4.1
Changed lines of the file:
@@
 Text Label 3950 2700 2    50   ~ 0
 RST
+$Comp
+L SamacSys_Parts:TAJB476M010TNJ C4
+U 1 1 60363F6C
+P 5300 3700
+F 0 "C4" V 5504 3830 50  0000 L CNN
+F 1 "TAJB476M010TNJ" V 5595 3830 50  0000 L CNN
+F 2 "CAPPM3528X210N" H 5650 3750 50  0001 L CNN
+F 3 "http://datasheets.avx.com/TAJ.pdf" H 5650 3650 50  0001 L CNN
+F 4 "Tantalum Capacitors - Solid SMD 10volts 47uF 20%" H 5650 3550 50  0001 L CNN "Description"
+F 5 "2.1" H 5650 3450 50  0001 L CNN "Height"
+F 6 "AVX" H 5650 3350 50  0001 L CNN "Manufacturer_Name"
+F 7 "TAJB476M010TNJ" H 5650 3250 50  0001 L CNN "Manufacturer_Part_Number"
+F 8 "581-TAJB476M010TNJ" H 5650 3150 50  0001 L CNN "Mouser Part Number"
+F 9 "https://www.mouser.co.uk/ProductDetail/AVX/TAJB476M010TNJ?qs=pYVYkI7xuRVorIKKgcxm0A%3D%3D" H 5650 3050 50  0001 L CNN "Mouser Price/Stock"
+F 10 "TAJB476M010TNJ" H 5650 2950 50  0001 L CNN "Arrow Part Number"
+F 11 "https://www.arrow.com/en/products/tajb476m010tnj/avx" H 5650 2850 50  0001 L CNN "Arrow Price/Stock"
+	1    5300 3700
+	0    1    1    0
+$EndComp
+Text Label 5300 4200 0    50   ~ 0
+GND
 $EndSCHEMATC

Commit message: Added 100nF decoupling capacitors between VCC and Ground of the ESP
Parts:
- added C?: 100nF, handsolder:C_0402_1005Metric_Pad0.74x0.62mm_HandSoldermod, symbol Device:C
Connections:
- net GND: now also C?.2
- net VCC: now also C?.1
Changed lines of the file:
@@
 Text Label 5300 4200 0    50   ~ 0
 GND
+$Comp
+L Device:C C?
+U 1 1 6036783B
+P 4900 3900
+F 0 "C?" H 5015 3946 50  0000 L CNN
+F 1 "100nF" H 5015 3855 50  0000 L CNN
+F 2 "handsolder:C_0402_1005Metric_Pad0.74x0.62mm_HandSoldermod" H 4938 3750 50  0001 C CNN
+F 3 "~" H 4900 3900 50  0001 C CNN
+	1    4900 3900
+	1    0    0    -1
+$EndComp
+Wire Wire Line
+	4900 3750 4900 3700
+Wire Wire Line
+	4900 3700 5300 3700
+Connection ~ 5300 3700
+Wire Wire Line
+	4900 4050 5150 4050
+Wire Wire Line
+	5150 4050 5150 4200
+Wire Wire Line
+	5150 4200 5300 4200
 $EndSCHEMATC
