File: button - AA [ORDERED]/button.sch (KiCad schematic (older format))
At the start: 20 parts, among them J1 Conn_01x06_Male, SW1 SW_Push, SW2 SW_Push, U1 TLV61224, U2 AP2112K-3.3, X1 ESP-12E

Commit message: turned around some of the LIPO connectors
Parts:
- U2: symbol Regulator_Linear:AP2112K-3.3 -> button-rescue:AP2112K-3.3-Regulator_Linear
Changed lines of the file:
@@
 	2750 4100 2800 4100
 $Comp
-L Regulator_Linear:AP2112K-3.3 U2
+L button-rescue:AP2112K-3.3-Regulator_Linear U2
 U 1 1 602F5FBE
 P 3600 5100

Commit message: added BOMs
Connections:
- net VCC: now also D1.2 (A); no longer D1.1 (K)
- net at R6.1: now also D1.1 (K); no longer D1.2 (A)
Other:
- moved on the sheet: D1
Changed lines of the file:
@@
 F 3 "~" H 6800 1450 50  0001 C CNN
 	1    6800 1450
-	0    1    1    0
+	0    -1   -1   0
 $EndComp
 Wire Wire Line
