File: button_timer_v1.2.1_lipo[TPL5111] - corrected/button_timer_v1.2.1_lipo.sch (KiCad schematic (older format))
At the start: 25 parts, among them J1 Conn_01x05_Female, SW1 SW_Push, SW2 SW_Push, U2 AP2112K-3.3, U3 TPL5111, X1 ESP-12E

Commit message: All Footprints corrected
Parts:
- removed X1: ESP-12E, handsolder:ESP-12Elesssilk, symbol button-timer-v1.2-rescue:ESP-12E-ardafruit-button-timer-rescue-button-timer-v1.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
- added X1: ESP-12E, handsolder:ESP-12Elesssilk, symbol ardafruit:ESP-12E
- D1: footprint LED_SMD:LED_1206_3216Metric_Castellated -> handsolder:LED_0805_2012Metric_Castellated_mod
- D2: footprint LED_SMD:LED_0805_2012Metric_Castellated -> handsolder:LED_1206_3216Metric_Castellated
Connections:
- net EN: now also X1.3 (CH_PD)
- net GND: now also X1.15 (GND)
- net GPIO0: now also X1.18 (GPIO0)
- net GPIO15: now also X1.16 (GPIO15)
- net GPIO2: now also X1.17 (GPIO2)
- net GPIO4: now also X1.19 (GPIO4)
- net GPIO5: now also X1.20 (GPIO5)
- net RST: now also X1.1 (RESET)
- net RX: now also X1.21 (RXD)
- net TX: now also X1.22 (TXD)
- net VCC: now also X1.8 (VCC)
Changed lines of the file:
@@
 $EndDescr
-$Comp
-L button-timer-v1.2-rescue:ESP-12E-ardafruit-button-timer-rescue-button-timer-v1.2-rescue-button-timer-v1.2-rescue-button-timer-v1.2-rescue-button-timer-v1.2-rescue X1
-U 1 1 602C0443
-P 6000 3400
-F 0 "X1" H 6000 3400 50  0001 C CNN
-F 1 "ESP-12E" H 6000 3400 50  0001 C CNN
-F 2 "handsolder:ESP-12Elesssilk" H 6000 3400 50  0001 C CNN
-F 3 "" H 6000 3400 50  0001 C CNN
-	1    6000 3400
-	1    0    0    -1
-$EndComp
 $Comp
 L button-timer-v1.2-rescue:Battery_Cell-Device-button-timer-rescue-button-timer-v1.2-rescue-button-timer-v1.2-rescue-button-timer-v1.2-rescue-button-timer-v1.2-rescue BT1
@@
 F 0 "D2" H 6743 4395 50  0000 C CNN
 F 1 "LED" H 6743 4486 50  0000 C CNN
-F 2 "LED_SMD:LED_0805_2012Metric_Castellated" H 6750 4650 50  0001 C CNN
+F 2 "handsolder:LED_1206_3216Metric_Castellated" H 6750 4650 50  0001 C CNN
 F 3 "~" H 6750 4650 50  0001 C CNN
 	1    6750 4650
@@
 F 0 "D1" V 1097 6328 50  0000 L CNN
 F 1 "LED" V 1188 6328 50  0000 L CNN
-F 2 "LED_SMD:LED_1206_3216Metric_Castellated" H 1150 6250 50  0001 C CNN
+F 2 "handsolder:LED_0805_2012Metric_Castellated_mod" H 1150 6250 50  0001 C CNN
 F 3 "~" H 1150 6250 50  0001 C CNN
 	1    1150 6250
@@
 Wire Wire Line
 	5050 3700 5300 3700
+Wire Wire Line
+	5050 4050 5050 4200
+Wire Wire Line
+	5050 4200 5300 4200
+$Comp
+L ardafruit:ESP-12E X1
+U 1 1 603C27E0
+P 6000 3400
+F 0 "X1" H 6000 3400 50  0001 C CNN
+F 1 "ESP-12E" H 6000 3400 50  0001 C CNN
+F 2 "handsolder:ESP-12Elesssilk" H 6000 3400 50  0001 C CNN
+F 3 "" H 6000 3400 50  0001 C CNN
+	1    6000 3400
+	1    0    0    -1
+$EndComp
 Connection ~ 5300 3700
-Wire Wire Line
-	5050 4050 5050 4200
-Wire Wire Line
-	5050 4200 5300 4200
 $EndSCHEMATC
