File: button v2- AAA - corrected/button - AAA.kicad_pcb (KiCad board)
At the start: 2 copper layers, 20.3 x 60.6 mm, 22 parts, among them J1 Conn_01x05_Female, SW1 SW_Push, SW2 SW_Push, U2 AP2112K-3.3, X1 ESP-12E

Commit message: :)
Other:
- rule pad_to_mask_clearance: 0.051 -> 0
