File: button v2_1 - AA [TPL5110]/button v2_1 - AA [TPL5110].kicad_pcb (KiCad board)
At the start: 2 copper layers, 20.3 x 69.5 mm, 27 parts, among them J1 Conn_01x06_Male, SW1 SW_Push, SW2 SW_Push, U1 TPL5110, U2 AP2112K-3.3, U3 TSM2323CX, X1 ESP-12E

Commit message: :)
Other:
- rule pad_to_mask_clearance: 0.051 -> 0
