File: button_timer v1.2.3_Coin_Cell[TPL5111] - corrected/button timer v1.2.3_Coin_Cell[TPL5111].kicad_pcb (KiCad board)
At the start: 2 copper layers, 21 x 47.8 mm, 27 parts, among them J1 Conn_01x05_Female, Q1 mmbt2222, SW1 SW_Push, SW2 SW_Push, U1 TPS61097A, U3 TPL5111, X1 ESP-12E

Commit message: :)
Other:
- rule pad_to_mask_clearance: 0.051 -> 0
