File: button_timer_v1.2.1_lipo[TPL5110] - corrected/button_timer_v1.2.1_lipo[TPL5110].kicad_pcb (KiCad board)
At the start: 2 copper layers, 21 x 41.7 mm, 26 parts, among them J1 Conn_01x05_Female, Q1 TSM2301ACX, SW1 SW_Push, SW2 SW_Push, U1 TPL5110, U2 AP2112K-3.3, X1 ESP-12E

Commit message: :)
Other:
- rule pad_to_mask_clearance: 0.051 -> 0
