File: button_v1.2.2_Coin_Cell[NO TIMER] -- corrected/button_v1.2.2_Coin_Cell.kicad_pcb (KiCad board)
At the start: 2 copper layers, 21 x 47.8 mm, 20 parts, among them J1 Conn_01x05_Female, SW1 SW_Push, SW2 SW_Push, U1 TPS61097A, X1 ESP-12E

Commit message: :)
Other:
- rule pad_to_mask_clearance: 0.051 -> 0
